Commit message: Update robot.urdf.xacro

File: robot_description/urdf/robot.urdf.xacro (robot description, xacro)
@@ -83,118 +83,4 @@
     </inertial>
   </link>
-  <!-- sick LiDAR 0 -->
-  <joint name="sick_lidar0_joint" type="fixed">
-    <parent link="base_link"/>
-    <child link="sick_lidar0"/>
-    <origin xyz="0.33 0.175 0.195722" rpy="0 0 0.7854"/>
-  </joint>
-  <link name="sick_lidar0">
-    <collision>
-      <origin xyz="0 0 0" rpy="0 0 0"/>
-      <geometry>
-        <mesh filename="package://robot_description/meshes/sick_s30b.stl" scale="0.01 0.01 0.01"/>
-      </geometry>
-    </collision>
-    <visual>
-      <origin xyz="0 0 0" rpy="0 0 0"/>
-      <geometry>
-        <mesh filename="package://robot_description/meshes/sick_s30b.stl" scale="0.01 0.01 0.01"/>
-      </geometry>
-      <material name="green"/>
-    </visual>
-    <inertial>
-      <origin xyz="0 0 0" rpy="0 0 0"/>
-      <mass value="1.2"/>
-      <inertia ixx="0.0001" ixy="0.0" ixz="0.0"
-	             iyy="0.0001" iyz="0.0"
-	             izz="0.0001"/>
-      </inertial>
-  </link>
-  <!-- sick LiDAR 1 -->
-  <joint name="sick_lidar1_joint" type="fixed">
-    <parent link="base_link"/>
-    <child link="sick_lidar1"/>
-    <origin xyz="-0.33 -0.175 0.195722" rpy="0 0 -2.35619"/>
-  </joint>
-  <link name="sick_lidar1">
-    <collision>
-      <origin xyz="0 0 0" rpy="0 0 0"/>
-      <geometry>
-        <mesh filename="package://robot_description/meshes/sick_s30b.stl" scale="0.01 0.01 0.01"/>
-      </geometry>
-    </collision>
-    <visual>
-      <origin xyz="0 0 0" rpy="0 0 0"/>
-      <geometry>
-        <mesh filename="package://robot_description/meshes/sick_s30b.stl" scale="0.01 0.01 0.01"/>
-      </geometry>
-      <material name="green"/>
-    </visual>
-    <inertial>
-      <origin xyz="0 0 0" rpy="0 0 0"/>
-      <mass value="1.2"/>
-      <inertia ixx="0.0001" ixy="0.0" ixz="0.0"
-	             iyy="0.0001" iyz="0.0"
-	             izz="0.0001"/>
-      </inertial>
-  </link>
-  <!-- kinect V2 -->
-  <joint name="kinect_v2_joint " type="fixed">
-    <parent link="base_link"/>
-    <child link="kinect_v2"/>
-    <origin xyz="0.297 -0.05 0.122015" rpy="0 0 0"/>
-    <axis xyz="0 0 1"/>
-  </joint>
-  <link name="kinect_v2">
-    <collision>
-      <origin xyz="0 0 0" rpy="0 0 0"/>
-      <geometry>
-	      <mesh filename="package://robot_description/meshes/kinect_v2.stl" scale="0.01 0.01 0.01"/>
-      </geometry>
-    </collision>
-    <visual>
-      <origin xyz="0 0 0" rpy="0 0 0"/>
-      <geometry>
-	      <mesh filename="package://robot_description/meshes/kinect_v2.stl" scale="0.01 0.01 0.01"/>
-      </geometry>
-      <material name="black"/>
-    </visual>
-    <inertial>
-      <origin xyz="0 0 0" rpy="0 0 0"/>
-      <mass value="0.5"/>
-      <inertia ixx="0.00005" ixy="0.0" ixz="0.0"
-	             iyy="0.00005" iyz="0.0"
-	             izz="0.00005"/>
-    </inertial>
-  </link>
-  <!-- IMU -->
-  <joint name="IMU_joint " type="fixed">
-    <parent link="base_link"/>
-    <child link="IMU_sensor"/>
-    <origin xyz="0 0 0.08" rpy="0 0 0"/>
-    <axis xyz="0 0 1"/>
-  </joint>
-  <link name="IMU_sensor">
-    <collision>
-      <origin xyz="0 0 0" rpy="0 0 0"/>
-      <geometry>
-	      <mesh filename="package://robot_description/meshes/IMU_sensor.stl" scale="0.01 0.01 0.01"/>
-      </geometry>
-    </collision>
-    <visual>
-      <origin xyz="0 0 0" rpy="0 0 0"/>
-      <geometry>
-	      <mesh filename="package://robot_description/meshes/IMU_sensor.stl" scale="0.01 0.01 0.01"/>
-      </geometry>
-      <material name="red"/>
-    </visual>
-    <inertial>
-      <origin xyz="0 0 0" rpy="0 0 0"/>
-      <mass value="0.5"/>
-      <inertia ixx="0.00005" ixy="0.0" ixz="0.0"
-	             iyy="0.00005" iyz="0.0"
-	            izz="0.00005"/>
-    </inertial>
-  </link>
   <!--zm robot LR wheel-->
   <xacro:wheel_v1 prefix="1" parent="base_link" origin_x="${wheel_after_L}" origin_y="${wheel_left_W}" rotation_x="${wheel_rotationx}">
@@ -400,16 +286,3 @@
   <xacro:roller_trans_v0 prefix="roller_4_8"/>
   <xacro:roller_trans_v0 prefix="roller_4_9"/>
-  <!-- ultrasound -->
-  <xacro:ultrasound prefix="1" parent="base_link" origin_x="${ul_left_front_x}" origin_y="${ul_left_front_y}"
-                                                     origin_z="${ul_hight}" rotation_z="${ul_front_rotation}">
-  </xacro:ultrasound>
-  <xacro:ultrasound prefix="2" parent="base_link" origin_x="${ul_right_front_x}" origin_y="${ul_right_front_y}"
-                                                     origin_z="${ul_hight}" rotation_z="${ul_front_rotation}">
-  </xacro:ultrasound>
-  <xacro:ultrasound prefix="3" parent="base_link" origin_x="${ul_left_rear_x}" origin_y="${ul_left_rear_y}"
-                                                     origin_z="${ul_hight}" rotation_z="${ul_rear_rotation}">
-  </xacro:ultrasound>
-  <xacro:ultrasound prefix="4" parent="base_link" origin_x="${ul_right_rear_x}" origin_y="${ul_right_rear_y}"
-                                                     origin_z="${ul_hight}" rotation_z="${ul_rear_rotation}">
-  </xacro:ultrasound>
 </robot>
